File: kicad/first.kicad_pcb (KiCad board)
At the start: 2 copper layers, 122 parts, among them J1 Conn_01x04_Pin, J2 USB_C_Receptacle_USB2.0_16P, J3 PJ-603, J4 PJ-603, J5 PJ-328A0-B, J6 PJ-328A0-B, J7 Conn_02x08_Odd_Even, Q5 MMUN2111LT1G, Q6 MMUN2111LT1G, Q7 MMBT3904, Q8 MMBT3904, SW1 SPST, SW2 RotaryEncoder_Switch_MP, SW3 RotaryEncoder_Switch_MP, SW4 RotaryEncoder_Switch_MP, SW5 MSS22D18G2 125, U1 STM32F407VETx, U2 CS4272, U3 TPS7A20xxxDBV, U4 OPA1678, U5 OPA1678, U6 OPA1678, U7 USBLC6-2SC6, Y2 16MHz

Commit message: aaaa
Parts:
- U2: moved to F.Cu
- moved U2 132.6 mm to (165.8, 99.0), turned to 180 degrees
- moved J1 132.1 mm to (195.5, 97.6), turned to 180 degrees
- moved C7 129.1 mm to (173.0, 106.8)
- moved C13 129.0 mm to (175.0, 117.0)
- moved U1 129.0 mm to (183.8, 109.3)
- moved C12 129.0 mm to (176.4, 118.4)
- moved C5 129.0 mm to (194.8, 109.5)
- moved C4 129.0 mm to (186.7, 119.8)
- moved C47 129.0 mm to (194.7, 111.9)
- moved Y2 129.0 mm to (173.8, 119.3)
- moved C10 128.9 mm to (182.8, 123.1), turned to 45 degrees
- moved C2 128.8 mm to (175.8, 115.0)
- moved C1 128.8 mm to (174.1, 114.0), turned to -135 degrees
- moved C46 128.7 mm to (187.8, 98.8)
- moved C11 128.7 mm to (178.5, 121.5)
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Connections:
- net /first/out1 renamed /first/D2
- net /first/out2 renamed /first/D3
- net /first/out3 renamed /first/D4
- net Net-(U1-VCAP_1) renamed /first/VCAP_1
- net Net-(U1-VCAP_2) renamed /first/VCAP_2
- net TIM2_CH1 renamed ENC1_TIM2_CH1
- net TIM2_CH2 renamed ENC1_TIM2_CH2
- net TIM3_CH1 renamed ENC2_TIM3_CH1
- net TIM3_CH2 renamed ENC2_TIM3_CH2
- C32 pad 2: Net-(U6A--) -> Net-(U6B--)
- C33 pad 2: Net-(U6A-+) -> Net-(U6B-+)
- C38 pad 2: Net-(U6B--) -> Net-(U6A--)
- C39 pad 2: Net-(U6B-+) -> Net-(U6A-+)
- J7 pad 10: GPIO2 -> GPIO4
- J7 pad 11: GPIO3 -> GPIO5
- J7 pad 12: GPIO4 -> GND
- J7 pad 13: GPIO5 -> USART3_RX
- J7 pad 14: GND -> USART3_TX
- J7 pad 3: USART3_TX -> SPI2_MISO
- J7 pad 4: USART3_RX -> SPI2_SCK
- J7 pad 6: SPI2_SCK -> SPI2_MOSI
- J7 pad 7: SPI2_MISO -> GPIO1
- J7 pad 8: SPI2_MOSI -> GPIO2
- J7 pad 9: GPIO1 -> GPIO3
- R27 pad 2: Net-(U6A--) -> Net-(U6B--)
- R29 pad 2: Net-(U6A-+) -> Net-(U6B-+)
- R37 pad 2: Net-(U6B--) -> Net-(U6A--)
- R39 pad 2: Net-(U6B-+) -> Net-(U6A-+)
- R5 pad 2: /first/I2C1_SDA -> /first/I2C3_SCL
- R6 pad 2: /first/I2C1_SCL -> /first/I2C3_SDA
- SW4 pad A: TIM4_CH1 -> ENC3_TIM1_CH1
- SW4 pad B: TIM4_CH2 -> ENC3_TIM1_CH2
- SW5 pad 1: /audio_IO/MIC_IN -> Net-(SW5-Pad1)
- SW5 pad 3: Net-(SW5-Pad3) -> /audio_IO/MIC_IN
- SW5 pad 4: Net-(C45-Pad1) -> Net-(SW5-Pad1)
- SW5 pad 6: Net-(SW5-Pad3) -> Net-(C45-Pad1)
- U1 pad 37: GPIO4 -> unconnected-(U1-PB2-Pad37)
- U1 pad 38: unconnected-(U1-PE7-Pad38) -> GPIO4
- U1 pad 40: unconnected-(U1-PE9-Pad40) -> ENC3_TIM1_CH1
- U1 pad 41: unconnected-(U1-PE10-Pad41) -> ENC3_SW
- U1 pad 42: unconnected-(U1-PE11-Pad42) -> ENC3_TIM1_CH2
- U1 pad 47: unconnected-(U1-PB10-Pad47) -> SPI2_SCK
- U1 pad 52: SPI2_SCK -> unconnected-(U1-PB13-Pad52)
- U1 pad 66: unconnected-(U1-PC9-Pad66) -> /first/I2C3_SDA
- U1 pad 67: unconnected-(U1-PA8-Pad67) -> /first/I2C3_SCL
- U1 pad 78: /first/I2S_CK -> unconnected-(U1-PC10-Pad78)
- U1 pad 79: /first/I2S_ext_SD -> unconnected-(U1-PC11-Pad79)
- U1 pad 80: /first/I2S_SD -> unconnected-(U1-PC12-Pad80)
- U1 pad 89: unconnected-(U1-PB3-Pad89) -> /first/I2S_CK
- U1 pad 90: unconnected-(U1-PB4-Pad90) -> /first/I2S_ext_SD
- U1 pad 91: ENC3_SW -> /first/I2S_SD
- U1 pad 92: TIM4_CH1 -> unconnected-(U1-PB6-Pad92)
- U1 pad 93: TIM4_CH2 -> unconnected-(U1-PB7-Pad93)
- U1 pad 95: /first/I2C1_SCL -> unconnected-(U1-PB8-Pad95)
- U1 pad 96: /first/I2C1_SDA -> unconnected-(U1-PB9-Pad96)
- U2 pad 11: /first/I2C1_SCL -> /first/I2C3_SCL
- U2 pad 12: /first/I2C1_SDA -> /first/I2C3_SDA
- U6 pad 1: Net-(C34-Pad1) -> Net-(C40-Pad1)
- U6 pad 7: Net-(C40-Pad1) -> Net-(C34-Pad1)
Routing:
- net VBUS: track 0.00 -> 82.0 mm
- net USART3_RX: track 0.00 -> 37.3 mm
- net /audio_IO/Left: track 0.00 -> 33.8 mm
- net USART3_TX: track 0.00 -> 31.8 mm
- net VQ23: track 0.00 -> 31.0 mm
- net /first/I2C3_SCL: track 0.00 -> 30.5 mm
- net GND: track 0.00 -> 27.9 mm
- net AOUTB+: track 0.00 -> 25.9 mm
- net AOUTB-: track 0.00 -> 25.9 mm
- net /first/I2S_SD: track 0.00 -> 23.8 mm
- net AOUTA+: track 0.00 -> 23.6 mm
- net AOUTA-: track 0.00 -> 23.6 mm
- net AIN_R: track 0.00 -> 23.2 mm
- net +3.3V: track 0.00 -> 22.4 mm
- net /audio_IO/Right: track 0.00 -> 21.2 mm
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Other:
- copper layers 2 -> 4

Commit message: aaa
Parts:
- moved R13 24.0 mm to (168.2, 119.0), turned to -90 degrees
- moved R12 21.5 mm to (166.8, 119.0), turned to -90 degrees
- moved R11 21.0 mm to (165.2, 119.0), turned to -90 degrees
- moved C11 20.4 mm to (195.7, 110.4)
- moved R7 14.7 mm to (172.8, 130.8)
- moved R1 12.8 mm to (171.8, 79.5), turned to 180 degrees
- moved R43 10.9 mm to (118.8, 114.3)
- moved R44 10.3 mm to (123.2, 114.6)
- moved Q6 10.1 mm to (126.5, 114.2)
- moved Q8 9.75 mm to (122.2, 111.9), turned to 180 degrees
- moved R45 9.27 mm to (125.2, 110.9), turned to 90 degrees
- moved R42 7.74 mm to (115.8, 113.2), turned to -90 degrees
- moved R3 6.24 mm to (193.5, 78.0), turned to 90 degrees
- moved R8 3.68 mm to (132.2, 117.2)
- moved R10 3.47 mm to (162.5, 117.2)
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Connections:
- J7 pad 10: GPIO4 -> GPIO1
- J7 pad 11: GPIO5 -> GPIO4
- J7 pad 12: GND -> GPIO3
- J7 pad 13: USART3_RX -> GND
- J7 pad 14: USART3_TX -> GPIO5
- J7 pad 7: GPIO1 -> USART2_RX
- J7 pad 8: GPIO2 -> USART2_TX
- J7 pad 9: GPIO3 -> GPIO2
- U1 pad 1: unconnected-(U1-PE2-Pad1) -> /first/D2
- U1 pad 2: unconnected-(U1-PE3-Pad2) -> /first/D3
- U1 pad 25: ENC1_SW -> USART2_TX
- U1 pad 26: unconnected-(U1-PA3-Pad26) -> USART2_RX
- U1 pad 3: unconnected-(U1-PE4-Pad3) -> /first/D4
- U1 pad 30: ENC2_SW -> unconnected-(U1-PA5-Pad30)
- U1 pad 39: unconnected-(U1-PE8-Pad39) -> GPIO5
- U1 pad 4: unconnected-(U1-PE5-Pad4) -> ENC1_SW
- U1 pad 41: ENC3_SW -> unconnected-(U1-PE10-Pad41)
- U1 pad 5: unconnected-(U1-PE6-Pad5) -> ENC2_SW
- U1 pad 55: USART3_TX -> unconnected-(U1-PD8-Pad55)
- U1 pad 56: USART3_RX -> unconnected-(U1-PD9-Pad56)
- U1 pad 59: /first/D2 -> unconnected-(U1-PD12-Pad59)
- U1 pad 60: /first/D3 -> unconnected-(U1-PD13-Pad60)
- U1 pad 61: /first/D4 -> unconnected-(U1-PD14-Pad61)
- U1 pad 62: GPIO5 -> unconnected-(U1-PD15-Pad62)
- U1 pad 7: unconnected-(U1-PC13-Pad7) -> ENC3_SW
Routing:
- net GND: track 27.9 -> 145.9 mm
- net GPIO1: track 0.00 -> 37.4 mm
- net USART3_RX: track 37.3 -> 0.00 mm
- net USART3_TX: track 31.8 -> 0.00 mm
- net +5VA: track 15.1 -> 42.0 mm
- net Net-(J4-Pad3): track 0.00 -> 25.9 mm
- net AOUT_L: track 0.00 -> 22.1 mm
- net GPIO4: track 0.00 -> 20.6 mm
- net /first/NRST: track 0.00 -> 19.4 mm
- net GPIO2: track 0.00 -> 19.3 mm
- net AOUT_R: track 0.00 -> 18.8 mm
- net GPIO5: track 0.00 -> 17.6 mm
- net GPIO3: track 0.00 -> 17.0 mm
- net USART2_RX: track 0.00 -> 16.3 mm
- net USART2_TX: track 0.00 -> 13.3 mm
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
Commit message: a
Parts:
- moved C41 2.25 mm to (148.0, 111.0)
- moved D3 1.77 mm to (147.0, 117.2)
- moved R9 1.77 mm to (147.0, 115.5)
- moved SW3 1.77 mm to (144.8, 134.5)
- moved D2 1.75 mm to (132.2, 117.2)
- moved D4 1.75 mm to (162.5, 117.2)
- moved R10 1.75 mm to (162.5, 115.5)
- moved R11 1.75 mm to (165.2, 117.3)
- moved R12 1.75 mm to (166.8, 117.3)
- moved R13 1.75 mm to (168.2, 117.2)
- moved R8 1.75 mm to (132.2, 115.5)
- moved SW2 1.75 mm to (129.8, 134.5)
- moved SW4 1.75 mm to (160.2, 134.5)
Changed lines of the file:
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@@
 	(footprint "Rotary_Encoder:RotaryEncoder_Alps_EC11E-Switch_Vertical_H20mm"
 		(layer "F.Cu")
-		(at 129.75 136.25 90)
+		(at 129.75 134.5 90)
 		(descr "Alps rotary encoder, EC11E... with switch, vertical shaft, http://www.alps.com/prod/info/E/HTML/Encoder/Incremental/EC11/EC11E15204A3.html")
 		(tags "rotary encoder")
@@
 	(footprint "Capacitor_SMD:CP_Elec_4x5.4"
 		(layer "F.Cu")
-		(at 148 113.25)
+		(at 148 111)
 		(descr "SMD capacitor, aluminum electrolytic, Panasonic A5 / Nichicon, 4.0x5.4mm")
 		(tags "capacitor electrolytic")
@@
 	(footprint "Resistor_SMD:R_0402_1005Metric"
 		(layer "F.Cu")
-		(at 147.25 117.25 180)
+		(at 147 115.5 180)
 		(descr "Resistor SMD 0402 (1005 Metric), square (rectangular) end terminal, IPC-7351 nominal, (Body size source: IPC-SM-782 page 72, https://www.pcb-3d.com/wordpress/wp-content/uploads/ipc-sm-782a_amendment_1_and_2.pdf)")
 		(tags "resistor")
@@
 	(footprint "Rotary_Encoder:RotaryEncoder_Alps_EC11E-Switch_Vertical_H20mm"
 		(layer "F.Cu")
-		(at 145 136.25 90)
+		(at 144.75 134.5 90)
 		(descr "Alps rotary encoder, EC11E... with switch, vertical shaft, http://www.alps.com/prod/info/E/HTML/Encoder/Incremental/EC11/EC11E15204A3.html")
 		(tags "rotary encoder")
@@
 	(footprint "Resistor_SMD:R_0402_1005Metric"
 		(layer "F.Cu")
-		(at 168.25 119 -90)
+		(at 168.25 117.25 -90)
 		(descr "Resistor SMD 0402 (1005 Metric), square (rectangular) end terminal, IPC-7351 nominal, (Body size source: IPC-SM-782 page 72, https://www.pcb-3d.com/wordpress/wp-content/uploads/ipc-sm-782a_amendment_1_and_2.pdf)")
 		(tags "resistor")
@@
 	(footprint "Resistor_SMD:R_0402_1005Metric"
 		(layer "F.Cu")
-		(at 166.75 119.009999 -90)
+		(at 166.75 117.259999 -90)
 		(descr "Resistor SMD 0402 (1005 Metric), square (rectangular) end terminal, IPC-7351 nominal, (Body size source: IPC-SM-782 page 72, https://www.pcb-3d.com/wordpress/wp-content/uploads/ipc-sm-782a_amendment_1_and_2.pdf)")
 		(tags "resistor")
@@
 	(footprint "LED_SMD:LED_0603_1608Metric"
 		(layer "F.Cu")
-		(at 162.5 119)
+		(at 162.5 117.25)
 		(descr "LED SMD 0603 (1608 Metric), square (rectangular) end terminal, IPC-7351 nominal, (Body size source: http://www.tortai-tech.com/upload/download/2011102023233369053.pdf)")
 		(tags "LED")
@@
 	(footprint "Rotary_Encoder:RotaryEncoder_Alps_EC11E-Switch_Vertical_H20mm"
 		(layer "F.Cu")
-		(at 160.25 136.25 90)
+		(at 160.25 134.5 90)
 		(descr "Alps rotary encoder, EC11E... with switch, vertical shaft, http://www.alps.com/prod/info/E/HTML/Encoder/Incremental/EC11/EC11E15204A3.html")
 		(tags "rotary encoder")
@@
 	(footprint "Resistor_SMD:R_0402_1005Metric"
 		(layer "F.Cu")
-		(at 162.509999 117.25 180)
+		(at 162.509999 115.5 180)
 		(descr "Resistor SMD 0402 (1005 Metric), square (rectangular) end terminal, IPC-7351 nominal, (Body size source: IPC-SM-782 page 72, https://www.pcb-3d.com/wordpress/wp-content/uploads/ipc-sm-782a_amendment_1_and_2.pdf)")
 		(tags "resistor")
@@
 	(footprint "LED_SMD:LED_0603_1608Metric"
 		(layer "F.Cu")
-		(at 132.25 119)
+		(at 132.25 117.25)
 		(descr "LED SMD 0603 (1608 Metric), square (rectangular) end terminal, IPC-7351 nominal, (Body size source: http://www.tortai-tech.com/upload/download/2011102023233369053.pdf)")
 		(tags "LED")
@@
 	(footprint "LED_SMD:LED_0603_1608Metric"
 		(layer "F.Cu")
-		(at 147.25 119)
+		(at 147 117.25)
 		(descr "LED SMD 0603 (1608 Metric), square (rectangular) end terminal, IPC-7351 nominal, (Body size source: http://www.tortai-tech.com/upload/download/2011102023233369053.pdf)")
 		(tags "LED")
@@
 	(footprint "Resistor_SMD:R_0402_1005Metric"
 		(layer "F.Cu")
-		(at 132.25 117.25 180)
+		(at 132.25 115.5 180)
 		(descr "Resistor SMD 0402 (1005 Metric), square (rectangular) end terminal, IPC-7351 nominal, (Body size source: IPC-SM-782 page 72, https://www.pcb-3d.com/wordpress/wp-content/uploads/ipc-sm-782a_amendment_1_and_2.pdf)")
 		(tags "resistor")
@@
 	(footprint "Resistor_SMD:R_0402_1005Metric"
 		(layer "F.Cu")
-		(at 165.25 119.009999 -90)
+		(at 165.25 117.259999 -90)
 		(descr "Resistor SMD 0402 (1005 Metric), square (rectangular) end terminal, IPC-7351 nominal, (Body size source: IPC-SM-782 page 72, https://www.pcb-3d.com/wordpress/wp-content/uploads/ipc-sm-782a_amendment_1_and_2.pdf)")
 		(tags "resistor")
@@
 	)
 	(segment
-		(start 146.462499 119)
-		(end 146.462499 117.527502)
+		(start 146.212499 117.25)
+		(end 146.212499 115.777502)
 		(width 0.3)
 		(layer "F.Cu")
@@
 	)
 	(segment
-		(start 146.462499 117.527502)
-		(end 146.740001 117.25)
+		(start 146.212499 115.777502)
+		(end 146.490001 115.5)
 		(width 0.3)
 		(layer "F.Cu")
@@
 	)
 	(segment
-		(start 168.25 119.509999)
-		(end 166.009999 121.75)
+		(start 168.25 117.759999)
+		(end 166.009999 120)
 		(width 0.3)
 		(layer "F.Cu")
@@
 	)
 	(segment
-		(start 166.009999 121.75)
-		(end 165.25 121.75)
+		(start 166.009999 120)
+		(end 165.25 120)
 		(width 0.3)
 		(layer "F.Cu")
@@
 	)
 	(segment
-		(start 161.712499 117.537501)
-		(end 162 117.25)
+		(start 161.712499 115.787501)
+		(end 162 115.5)
 		(width 0.3)
 		(layer "F.Cu")
@@
 	)
 	(segment
-		(start 161.712499 119)
-		(end 161.712499 117.537501)
+		(start 161.712499 117.25)
+		(end 161.712499 115.787501)
 		(width 0.3)
 		(layer "F.Cu")
@@
 	)
 	(segment
-		(start 131.462499 119)
-		(end 131.462499 117.527502)
+		(start 131.462499 117.25)
+		(end 131.462499 115.777502)
 		(width 0.3)
 		(layer "F.Cu")
@@
 	)
 	(segment
-		(start 131.462499 117.527502)
-		(end 131.740001 117.25)
+		(start 131.462499 115.777502)
+		(end 131.740001 115.5)
 		(width 0.3)
 		(layer "F.Cu")
