File: kicad/first.kicad_pcb (KiCad board)
At the start: 4 copper layers, 122 parts, among them J1 Conn_01x04_Pin, J2 USB_C_Receptacle_USB2.0_16P, J3 PJ-603, J4 PJ-603, J5 PJ-328A0-B, J6 PJ-328A0-B, J7 Conn_02x08_Odd_Even, Q5 MMUN2111LT1G, Q6 MMUN2111LT1G, Q7 MMBT3904, Q8 MMBT3904, SW1 SPST, SW2 RotaryEncoder_Switch_MP, SW3 RotaryEncoder_Switch_MP, SW4 RotaryEncoder_Switch_MP, SW5 MSS22D18G2 125, U1 STM32F407VETx, U2 CS4272, U3 TPS7A20xxxDBV, U4 OPA1678, U5 OPA1678, U6 OPA1678, U7 USBLC6-2SC6, Y2 16MHz

Commit message: aaa
Connections:
- net /audio_IO/Left renamed /audio_io/Left
- net /audio_IO/MIC_IN renamed /audio_io/MIC_IN
- net /audio_IO/Right renamed /audio_io/Right
Routing:
- net GND: track 145.9 -> 38.4 mm
- net VBUS: track 85.1 -> 77.1 mm
- net +3.3V: track 27.7 -> 22.1 mm
- net SPI2_MISO: track 5.58 -> 1.87 mm
- net SPI2_MOSI: track 4.76 -> 1.25 mm
- net +5VA: track 42.0 -> 39.7 mm
- net +3.3VA: track 4.81 -> 2.90 mm

Commit message: moved to hierarchical sheets
Connections:
- net /audio_io/Left renamed /audio_conditioning/audio_io/Left
- net /audio_io/MIC_IN renamed /audio_conditioning/audio_io/MIC_IN
- net /audio_io/Right renamed /audio_conditioning/audio_io/Right
- net /first/BOOT0 renamed /BOOT0
- net /first/D2 renamed /D2
- net /first/D3 renamed /D3
- net /first/D4 renamed /D4
- net /first/HSE_IN renamed /HSE_IN
- net /first/HSE_OUT renamed /HSE_OUT
- net /first/I2C3_SCL renamed /I2C3_SCL
- net /first/I2C3_SDA renamed /I2C3_SDA
- net /first/I2S_CK renamed /I2S_CK
- net /first/I2S_MCK renamed /I2S_MCK
- net /first/I2S_SD renamed /I2S_SD
- net /first/I2S_WS renamed /I2S_WS
- net /first/I2S_ext_SD renamed /I2S_ext_SD
- net /first/NRST renamed /NRST
- net /first/PWR_LED_K renamed /PWR_LED_K
- net /first/SWCLK renamed /SWCLK
- net /first/SWDIO renamed /SWDIO
- net /first/USB_D+ renamed /USB_D+
- net /first/USB_D- renamed /USB_D-
- net /first/VCAP_1 renamed /VCAP_1
- net /first/VCAP_2 renamed /VCAP_2
- net AINA renamed /AINA
- net AINB renamed /AINB
- net AIN_L renamed /audio_conditioning/AIN_L
- net AIN_R renamed /audio_conditioning/AIN_R
- net AMUTEC renamed /AMUTEC
- net AOUTA+ renamed /AOUTA+
- net AOUTA- renamed /AOUTA-
- net AOUTB+ renamed /AOUTB+
- net AOUTB- renamed /AOUTB-
- net AOUT_L renamed /audio_conditioning/AOUT_L
- net AOUT_R renamed /audio_conditioning/AOUT_R
- net BMUTEC renamed /BMUTEC
- net VQ1 renamed /VQ1
- net VQ23 renamed /VQ23

Commit message: net classes
Connections:
- net GPIO1 renamed /GPIO1
- net GPIO2 renamed /GPIO2
- net GPIO3 renamed /GPIO3
- net GPIO4 renamed /GPIO4
- net GPIO5 renamed /GPIO5
- net SPI2_MISO renamed /SPI2_MISO
- net SPI2_MOSI renamed /SPI2_MOSI
- net SPI2_SCK renamed /SPI2_SCK
- net USART2_RX renamed /USART2_RX
- net USART2_TX renamed /USART2_TX
Routing:
- net /SPI2_SCK: track 14.2 -> 0.00 mm
- net /SPI2_MISO: track 1.87 -> 0.00 mm
- net /SWCLK: track 1.73 -> 0.00 mm
- net /SPI2_MOSI: track 1.25 -> 0.00 mm

Commit message: bla
Parts:
- added FID1: Fiducial, Fiducial:Fiducial_1mm_Mask3mm, F.Cu at (92.8, 76.0)
- added FID2: Fiducial, Fiducial:Fiducial_1mm_Mask3mm, F.Cu at (196.8, 79.2)
- added FID3: Fiducial, Fiducial:Fiducial_1mm_Mask3mm, F.Cu at (102.5, 132.8)
Routing:
- added copper zone on In1.Cu, net GND
Other:
- board outline added: 112.8 x 64.2 mm
